File: stellar/left/backlight.kicad_sch (KiCad schematic)
At the start: 31 parts

Commit message: [pcb] moved to 'left' folder
Other:
- company: (none) -> Robo productions
- title: (none) -> LED key backlight
Changed lines of the file:
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@@
 	(generator_version "8.0")
 	(paper "A4")
+	(title_block
+		(title "LED key backlight")
+		(date "2024-11-18")
+		(rev "v0.99")
+		(company "Robo productions")
+	)
 	(no_connect
 		(at 154.94 165.1)
