File: stellar/left/keymatrix.kicad_sch (KiCad schematic)
At the start: 50 parts, among them SW1 SW_Push_45deg, SW10 SW_Push_45deg, SW11 SW_Push_45deg, SW12 SW_Push_45deg, SW13 SW_Push_45deg, SW14 SW_Push_45deg, SW15 SW_Push_45deg, SW16 SW_Push_45deg, SW17 SW_Push_45deg, SW18 SW_Push_45deg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

Commit message: [pcb] moved to 'left' folder
Other:
- company: (none) -> Robo productions
- title: (none) -> Key matrix
Changed lines of the file:
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@@
 	(generator_version "8.0")
 	(paper "A4")
+	(title_block
+		(title "Key matrix")
+		(date "2024-11-18")
+		(rev "v0.99")
+		(company "Robo productions")
+	)
 	(junction
 		(at 165.1 124.46)
