File: stellar/left/stellar.kicad_pcb (KiCad board)
At the start: 2 copper layers, 158 x 119.2 mm, 100 parts, among them J1 Battery+, J2 Battery, J3 Battery-, J4 OLED, SW1 SW_Push_45deg, SW10 SW_Push_45deg, SW11 SW_Push_45deg, SW12 SW_Push_45deg, SW13 SW_Push_45deg, SW14 SW_Push_45deg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

Commit message: [pcb] moved to 'left' folder
Routing:
- net GND: vias 90 -> 95
Changed lines of the file:
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@@
+	)
+	(via
+		(at 147.4031 117.3236)
+		(size 0.4)
+		(drill 0.3)
+		(layers "F.Cu" "B.Cu")
+		(free yes)
+		(net 2)
 	)
 	(via
@@
 	)
 	(via
+		(at 147.4031 119.8236)
+		(size 0.4)
+		(drill 0.3)
+		(layers "F.Cu" "B.Cu")
+		(free yes)
+		(net 2)
+	)
+	(via
 		(at 207.4031 122.3236)
 		(size 0.4)
@@
 	)
 	(via
+		(at 149.9031 117.3236)
+		(size 0.4)
+		(drill 0.3)
+		(layers "F.Cu" "B.Cu")
+		(free yes)
+		(net 2)
+	)
+	(via
 		(at 137.4031 127.3236)
 		(size 0.4)
@@
 		(size 0.4)
 		(drill 0.3)
+		(layers "F.Cu" "B.Cu")
+		(free yes)
+		(net 2)
+	)
+	(via
+		(at 152.4031 117.3236)
+		(size 0.4)
+		(drill 0.3)
+		(layers "F.Cu" "B.Cu")
+		(free yes)
+		(net 2)
+	)
+	(via
+		(at 149.9031 119.8236)
+		(size 0.4)
+		(drill 0.3)

Commit message: [pcb] right half layout done
Routing:
- net GND: track 6.59 -> 0.00 mm
Other:
- board size 158 x 119.2 mm -> 158.8 x 119.9 mm
Changed lines of the file:
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@@
 		(tags "SOD-123")
 		(property "Reference" "D3"
-			(at 0 -2 -90)
+			(at 0 -2 90)
 			(unlocked yes)
-			(layer "F.SilkS")
+			(layer "B.SilkS")
 			(effects
 				(font
@@
 					(thickness 0.15)
 				)
+				(justify mirror)
 			)
 		)
@@
 		(tags "SOD-123")
 		(property "Reference" "D1"
-			(at 0 -2 -85)
+			(at 0 -2 95)
 			(unlocked yes)
 			(layer "B.SilkS")
@@
 		(at 138.048634 55.09784)
 		(property "Reference" "LED8"
-			(at 0 -2.5 180)
+			(at 0 -2.5 0)
 			(unlocked yes)
 			(layer "B.SilkS")
@@
 		(layer "Edge.Cuts")
 	)
+	(gr_arc
+		(start 216.76074 153.017301)
+		(mid 216.425316 153.178702)
+		(end 216.071279 153.063738)
+		(stroke
+			(width 0.15)
+			(type default)
+		)
+		(layer "Edge.Cuts")
+	)
 	(gr_line
 		(start 147.048119 37.775693)
-		(end 147.048119 33.789437)
+		(end 147.048119 33.790685)
 		(stroke
 			(width 0.149999)
@@
 		(layer "Edge.Cuts")
 	)
-	(gr_arc
-		(start 216.003747 152.363444)
-		(mid 215.683152 152.553935)
-		(end 215.319898 152.469586)
-		(stroke
-			(width 0.15)
-			(type default)
-		)
-		(layer "Edge.Cuts")
-	)
 	(gr_line
 		(start 68.867349 98.78692)
@@
 	)
 	(gr_arc
-		(start 68.411717 99.307799)
+		(start 68.411716 99.307785)
 		(mid 68.528175 98.9636)
-		(end 68.867349 98.78692)
+		(end 68.867349 98.786924)
 		(stroke
 			(width 0.15)
@@
 	)
 	(gr_arc
-		(start 77.204478 40.865824)
+		(start 77.204478 40.685611)
 		(mid 78.050165 38.686474)
 		(end 80.203123 37.775693)
@@
 	)
 	(gr_line
-		(start 69.80422 115.271113)
-		(end 68.411717 99.307799)
+		(start 227.01335 140.769257)
+		(end 216.76074 153.017301)
 		(stroke
 			(width 0.149999)
@@
 	)
 	(gr_line
-		(start 77.203123 129.282646)
+		(start 69.804188 115.270751)
+		(end 68.411716 99.307785)
+		(stroke
+			(width 0.149999)
+			(type solid)
+			(color 0 253 11 1)
+		)
+		(layer "Edge.Cuts")
+	)
+	(gr_line
+		(start 77.203123 129.283208)
 		(end 77.203123 115.125003)
 		(stroke
@@
 	)
 	(gr_line
+		(start 215.541803 130.462914)
+		(end 227.001906 140.04156)
+		(stroke
+			(width 0.149999)
+			(type solid)
+			(color 0 253 11 1)
+		)
+		(layer "Edge.Cuts")
+	)
+	(gr_line
 		(start 80.203123 132.29643)
-		(end 80.203123 132.293596)
+		(end 80.203123 132.293594)
 		(stroke
 			(width 0.149999)
@@
 	)
 	(gr_line
-		(start 226.2831 140.0836)
-		(end 216.003747 152.363444)
+		(start 216.071339 153.063665)
+		(end 208.751032 146.957545)
 		(stroke
 			(width 0.149999)
@@
 	(gr_line
 		(start 147.048119 37.775693)
-		(end 212.473835 37.775693)
+		(end 212.609765 37.775693)
 		(stroke
 			(width 0.149999)
@@
 	)
 	(gr_arc
-		(start 146.5495 33.327153)
+		(start 146.5496 33.327153)
 		(mid 146.9031 33.4736)
-		(end 147.048119 33.789437)
+		(end 147.048119 33.790685)
 		(stroke
 			(width 0.15)
@@
 	)
 	(gr_line
-		(start 146.5495 33.327153)
-		(end 129.483599 33.327153)
+		(start 146.5496 33.327153)
+		(end 129.602601 33.327153)
 		(stroke
 			(width 0.149999)
@@
 	(gr_line
 		(start 77.204478 98.052917)
-		(end 77.204478 40.865824)
+		(end 77.204478 40.685611)
 		(stroke
 			(width 0.149999)
@@
 	)
 	(gr_arc
-		(start 80.203123 132.293596)
+		(start 80.203123 132.293594)
 		(mid 78.081803 131.414923)
-		(end 77.203123 129.282646)
+		(end 77.203123 129.283208)
 		(stroke
 			(width 0.15)
@@
 	)
 	(gr_line
-		(start 215.319898 152.469586)
-		(end 208.747506 146.953748)
-		(stroke
-			(width 0.149999)
-			(type solid)
-			(color 0 253 11 1)
-		)
-		(layer "Edge.Cuts")
-	)
-	(gr_line
 		(start 189.952365 136.811725)
 		(end 191.298469 137.182647)
@@
 		(start 129.0431 33.8236)
 		(mid 129.189547 33.470047)
-		(end 129.483599 33.327153)
+		(end 129.602601 33.327153)
 		(stroke
 			(width 0.15)
@@
 	)
 	(gr_arc
-		(start 70.325099 115.726745)
+		(start 70.325113 115.726744)
 		(mid 69.9731 115.6036)
-		(end 69.80422 115.271113)
+		(end 69.804226 115.270748)
 		(stroke
 			(width 0.15)
@@
 	)
 	(gr_arc
-		(start 212.473835 37.775693)
+		(start 212.609765 37.775693)
 		(mid 214.663123 38.653603)
 		(end 215.541803 40.774923)
@@
 		(layer "Edge.Cuts")
 	)
-	(gr_line
-		(start 146.0531 133.8236)
-		(end 146.0531 132.29643)
+	(gr_arc
+		(start 227.001906 140.04156)
+		(mid 227.158871 140.334124)
+		(end 227.01335 140.769257)
 		(stroke
-			(width 0.149999)
-			(type solid)
-			(color 0 253 11 1)
+			(width 0.15)
+			(type default)
 		)
 		(layer "Edge.Cuts")
 	)
 	(gr_line
-		(start 215.541803 130.462914)
-		(end 226.1831 139.3936)
+		(start 146.0531 133.8236)
+		(end 146.0531 132.29643)
 		(stroke
 			(width 0.149999)
@@
 		(layer "Edge.Cuts")
 	)
-	(gr_arc
-		(start 226.1831 139.3936)
-		(mid 226.373591 139.714195)
-		(end 226.289242 140.077449)
-		(stroke
-			(width 0.15)
-			(type default)
-		)
-		(layer "Edge.Cuts")
-	)
 	(gr_line
 		(start 185.406132 135.855228)
@@
 	(gr_line
 		(start 77.203123 115.125003)
-		(end 70.325099 115.726745)
+		(end 70.325113 115.726744)
 		(stroke
 			(width 0.149999)
@@
 		(net 2)
 	)
-	(segment
-		(start 101.449095 129.527605)
-		(end 103.3231 127.6536)
-		(width 0.5)
-		(layer "B.Cu")
-		(net 2)
-	)
-	(segment
-		(start 103.827105 127.677605)
-		(end 105.692802 127.677605)
-		(width 0.5)
-		(layer "B.Cu")
-		(net 2)
-	)
-	(segment
-		(start 99.892802 129.527605)
-		(end 101.449095 129.527605)
-		(width 0.5)
-		(layer "B.Cu")
-		(net 2)
-	)
-	(segment
-		(start 103.8031 127.6536)
-		(end 103.827105 127.677605)
-		(width 0.5)
-		(layer "B.Cu")
-		(net 2)
-	)
-	(segment
-		(start 103.3231 127.6536)
-		(end 103.8031 127.6536)
-		(width 0.5)
-		(layer "B.Cu")
-		(net 2)
-	)

Commit message: [pcb] final version, maybe
Routing:
- net GND: vias 95 -> 79
