File: stellar/left/stellar.kicad_pcb (KiCad board)
At the start: 2 copper layers, 158.8 x 119.9 mm, 100 parts, among them J1 Battery+, J2 Battery, J3 Battery-, J4 OLED, SW1 SW_Push_45deg, SW10 SW_Push_45deg, SW11 SW_Push_45deg, SW12 SW_Push_45deg, SW13 SW_Push_45deg, SW14 SW_Push_45deg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

Commit message: [pcb] fixed logo and added J1 con 3D model
Parts:
- J2: footprint Connector_JST:JST_PH_S2B-PH-SM4-TB_1x02-1MP_P2.00mm_Horizontal -> Stellarlib:JST_PH_S2B-PH-SM4-TB_1x02-1MP_P2.00mm_Horizontal
Routing:
- net +3V3: track 712.5 -> 711.5 mm
