File: stellar/left/stellar.kicad_sch (KiCad schematic)
At the start: 19 parts, among them J1 Battery+, J2 Battery, J3 Battery-, J4 OLED, U1 Pro Micro NRF52840

Commit message: [pcb] moved to 'left' folder
Other:
- company: (none) -> Robo productions
- title: (none) -> Stellar left halve
Changed lines of the file:
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@@
 	(generator_version "8.0")
 	(paper "A4")
+	(title_block
+		(title "Stellar left halve")
+		(date "2024-11-18")
+		(rev "v0.99")
+		(company "Robo productions")
+	)
 	(junction
 		(at 256.54 57.15)

Commit message: [pcb] fixed logo and added J1 con 3D model
Parts:
- J2: footprint Connector_JST:JST_PH_S2B-PH-SM4-TB_1x02-1MP_P2.00mm_Horizontal -> Stellarlib:JST_PH_S2B-PH-SM4-TB_1x02-1MP_P2.00mm_Horizontal
Changed lines of the file:
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@@
 			)
 		)
-		(property "Footprint" "Connector_JST:JST_PH_S2B-PH-SM4-TB_1x02-1MP_P2.00mm_Horizontal"
+		(property "Footprint" "Stellarlib:JST_PH_S2B-PH-SM4-TB_1x02-1MP_P2.00mm_Horizontal"
 			(at 264.16 57.15 0)
 			(effects
